Commit message: 新增机器人模型与 Gazebo 启动配置

File: robot_description/rviz/robot.urdf.xacro (robot description, xacro)
@@ -26,4 +26,21 @@
             <origin xyz="0 0 0" rpy="1.5708 0 0"/>
         </visual>
+        <collision>
+            <origin xyz="0 0 0" rpy="1.5708 0 0"/>
+            <geometry>
+                <cylinder radius="0.1" length="0.05"/>
+            </geometry>
+        </collision>
+        <inertial>
+            <origin xyz="0 0 0"/>
+            <mass value="0.5"/>
+            <inertia
+                ixx="0.00135417"
+                ixy="0"
+                ixz="0"
+                iyy="0.0025"
+                iyz="0"
+                izz="0.00135417"/>
+        </inertial>
     </link>
     <joint name="left_wheel_joint" type="continuous">
@@ -40,4 +57,21 @@
             <origin xyz="0 0 0" rpy="1.5708 0 0"/>
         </visual>
+        <collision>
+            <origin xyz="0 0 0" rpy="1.5708 0 0"/>
+            <geometry>
+                <cylinder radius="0.1" length="0.05"/>
+            </geometry>
+        </collision>
+        <inertial>
+            <origin xyz="0 0 0"/>
+            <mass value="0.5"/>
+            <inertia
+                ixx="0.00135417"
+                ixy="0"
+                ixz="0"
+                iyy="0.0025"
+                iyz="0"
+                izz="0.00135417"/>
+        </inertial>
     </link>
     <joint name="right_wheel_joint" type="continuous">
