Commit message: 重构 ROS 2 工作区包结构

File: src/robot_description/urdf/base.xacro (robot description, xacro)
@@ -1,4 +1,4 @@
 <?xml version="1.0"?>
-<robot xmlns:xacro="http://www.ros.org/wiki/xacro" name="robot_base">
+<robot xmlns:xacro="http://www.ros.org/wiki/xacro">
     <link name="base_link">
         <visual>
@@ -21,8 +21,8 @@
     <link name="left_wheel_link">
         <visual>
+            <origin xyz="0 0 0" rpy="1.5708 0 0"/>
             <geometry>
                 <cylinder radius="0.1" length="0.05"/>
             </geometry>
-            <origin xyz="0 0 0" rpy="1.5708 0 0"/>
         </visual>
         <collision>
@@ -52,8 +52,8 @@
     <link name="right_wheel_link">
         <visual>
+            <origin xyz="0 0 0" rpy="1.5708 0 0"/>
             <geometry>
                 <cylinder radius="0.1" length="0.05"/>
             </geometry>
-            <origin xyz="0 0 0" rpy="1.5708 0 0"/>
         </visual>
         <collision>
